Commit message: added launchfile to have the robot in isaac, controller are just for testing

File: config/lekiwi.ros2_control.xacro (robot description, xacro)
@@ -6,10 +6,13 @@
                 <xacro:if value="${use_fake_hardware}">
                     <plugin>mock_components/GenericSystem</plugin>
+                    <param name="fake_sensor_commands">false</param>
+                    <param name="state_following_offset">0.0</param>
+                    <param name="calculate_dynamics">true</param>
                 </xacro:if>
                 <xacro:unless value="${use_fake_hardware}">
-                    <plugin>lekiwi_hardware/LeKiwiInterface</plugin>
-                    <param name="use_serial">true</param>
-                    <param name="serial_port">/dev/ttyUSB0</param>
-                    <param name="serial_baudrate">1000000</param>
+                    <plugin>joint_state_topic_hardware_interface/JointStateTopicSystem</plugin>
+                    <param name="joint_commands_topic">/topic_based_joint_commands</param>
+                    <param name="joint_states_topic">/topic_based_joint_states</param>
+                    <param name="sum_wrapped_joint_states">true</param>
                 </xacro:unless>
             </hardware>
@@ -20,4 +23,5 @@
                 </state_interface>
                 <state_interface name="velocity"/>
+                <state_interface name="effort"/>
                 <param name="motor_id">7</param>
                 <param name="direction">-1</param>
@@ -30,4 +34,5 @@
                 </state_interface>
                 <state_interface name="velocity"/>
+                <state_interface name="effort"/>
                 <param name="motor_id">8</param>
                 <param name="direction">-1</param>
@@ -40,8 +45,63 @@
                 </state_interface>
                 <state_interface name="velocity"/>
+                <state_interface name="effort"/>
                 <param name="motor_id">9</param>
                 <param name="direction">-1</param>
                 <param name="control_mode">velocity</param>
             </joint>
+            <joint name="STS3215_03a_v1_Revolute_45">
+                <command_interface name="position"/>
+                <state_interface name="position">
+                  <param name="initial_value">0</param>
+                </state_interface>
+                <state_interface name="velocity"/>
+                <state_interface name="effort"/>
+                <param name="control_mode">position</param>
+            </joint>
+            <joint name="STS3215_03a_v1_1_Revolute_49">
+                <command_interface name="position"/>
+                <state_interface name="position">
+                  <param name="initial_value">0</param>
+                </state_interface>
+                <state_interface name="velocity"/>
+                <state_interface name="effort"/>
+                <param name="control_mode">position</param>
+            </joint>
+            <joint name="STS3215_03a_v1_2_Revolute_51">
+                <command_interface name="position"/>
+                <state_interface name="position">
+                  <param name="initial_value">0</param>
+                </state_interface>
+                <state_interface name="velocity"/>
+                <state_interface name="effort"/>
+                <param name="control_mode">position</param>
+            </joint>
+            <joint name="STS3215_03a_v1_3_Revolute_53">
+                <command_interface name="position"/>
+                <state_interface name="position">
+                  <param name="initial_value">0</param>
+                </state_interface>
+                <state_interface name="velocity"/>
+                <state_interface name="effort"/>
+                <param name="control_mode">position</param>
+            </joint>
+            <joint name="STS3215_03a_Wrist_Roll_v1_Revolute_55">
+                <command_interface name="position"/>
+                <state_interface name="position">
+                  <param name="initial_value">0</param>
+                </state_interface>
+                <state_interface name="velocity"/>
+                <state_interface name="effort"/>
+                <param name="control_mode">position</param>
+            </joint>
+            <joint name="STS3215_03a_v1_4_Revolute_57">
+                <command_interface name="position"/>
+                <state_interface name="position">
+                  <param name="initial_value">0</param>
+                </state_interface>
+                <state_interface name="velocity"/>
+                <state_interface name="effort"/>
+                <param name="control_mode">position</param>
+            </joint>
         </ros2_control>
   </xacro:macro>

File: urdf/lekiwi.urdf (robot description, URDF)
Before this commit: robot LeKiwi, 46 links, 45 joints
Joints:
- removed joint STS3215_03a-v1-1_Revolute-49
- removed joint STS3215_03a-v1-2_Revolute-51
- removed joint STS3215_03a-v1-3_Revolute-53
- removed joint STS3215_03a-v1-4_Revolute-57
- removed joint STS3215_03a-v1_Revolute-45
- removed joint STS3215_03a_Wrist_Roll-v1_Revolute-55
- added joint STS3215_03a_Wrist_Roll_v1_Revolute_55: type revolute, parent STS3215_03a_Wrist_Roll-v1, child Wrist_Roll_08c-v1, origin xyz=-0.028999999999999998 0.00810632 0.006869499999999995 rpy=3.141592653589793 -0.0 0.0, axis 0.0 0.42261799999999994 -0.9063079999999999, limit lower=-3.14159 upper=3.14159 effort=10.0 velocity=5.0
- added joint STS3215_03a_v1_1_Revolute_49: type revolute, parent STS3215_03a-v1-1, child SO_ARM100_08k_116_Square-v1, origin xyz=0.0346 0.010249999999999987 -0.032799999999999975 rpy=3.141592653589793 1.7181275903033976e-32 -3.1373434374976504e-48, axis 1.0 0.0 0.0, limit lower=-3.14159 upper=3.14159 effort=10.0 velocity=5.0
- added joint STS3215_03a_v1_2_Revolute_51: type revolute, parent STS3215_03a-v1-2, child SO_ARM100_08k_Mirror-v1, origin xyz=0.0346 -0.013069710000000002 0.03178184000000002 rpy=-6.842277657836021e-49 -3.4512664603419266e-31 -1.3877787807814457e-17, axis 1.0 0.0 0.0, limit lower=-3.14159 upper=3.14159 effort=10.0 velocity=5.0
- added joint STS3215_03a_v1_3_Revolute_53: type revolute, parent STS3215_03a-v1-3, child Wrist_Roll_Pitch_08i-v1, origin xyz=0.0346 -0.03408158 0.004398620000000015 rpy=3.1415926535897922 9.860761315262648e-32 -9.503163413661107e-47, axis 1.0 0.0 9.860761315262648e-32, limit lower=-3.14159 upper=3.14159 effort=10.0 velocity=5.0
- added joint STS3215_03a_v1_4_Revolute_57: type revolute, parent STS3215_03a-v1-4, child Moving_Jaw_08d-v1, origin xyz=-0.032799999999999996 -0.023912249999999986 0.027026410000000018 rpy=-1.5707963267948968 3.944304526105059e-31 -1.9721522630525295e-31, axis -2.74128770133849e-31 -0.9063079999999999 -0.422618, limit lower=-3.14159 upper=3.14159 effort=10.0 velocity=5.0
- added joint STS3215_03a_v1_Revolute_45: type revolute, parent STS3215_03a-v1, child Rotation_Pitch_08i-v1, origin xyz=-0.010250000000000084 0.03459999999999999 -0.032799999999999996 rpy=1.5707963267948966 -2.781046729970605e-32 3.94430452610506e-31, axis -3.944304526105059e-31 3.944304526105059e-31 1.0, limit lower=-3.14159 upper=3.14159 effort=10.0 velocity=5.0

Commit message: getting commands to wheel. cmd_vel to joint commands needs fix

File: config/lekiwi.ros2_control.xacro (robot description, xacro)
@@ -17,37 +17,4 @@
                 </xacro:unless>
             </hardware>
-            <joint name="joint7">
-                <command_interface name="velocity"/>
-                <state_interface name="position">
-                  <param name="initial_value">0</param>
-                </state_interface>
-                <state_interface name="velocity"/>
-                <state_interface name="effort"/>
-                <param name="motor_id">7</param>
-                <param name="direction">-1</param>
-                <param name="control_mode">velocity</param>
-            </joint>
-            <joint name="joint8">
-                <command_interface name="velocity"/>
-                <state_interface name="position">
-                  <param name="initial_value">0</param>
-                </state_interface>
-                <state_interface name="velocity"/>
-                <state_interface name="effort"/>
-                <param name="motor_id">8</param>
-                <param name="direction">-1</param>
-                <param name="control_mode">velocity</param>
-            </joint>
-            <joint name="joint9">
-                <command_interface name="velocity"/>
-                <state_interface name="position">
-                  <param name="initial_value">0</param>
-                </state_interface>
-                <state_interface name="velocity"/>
-                <state_interface name="effort"/>
-                <param name="motor_id">9</param>
-                <param name="direction">-1</param>
-                <param name="control_mode">velocity</param>
-            </joint>
             <joint name="STS3215_03a_v1_Revolute_45">
                 <command_interface name="position"/>
@@ -104,4 +71,31 @@
                 <param name="control_mode">position</param>
             </joint>
+            <joint name="joint7">
+                <command_interface name="velocity"/>
+                <state_interface name="position">
+                  <param name="initial_value">0</param>
+                </state_interface>
+                <state_interface name="velocity"/>
+                <state_interface name="effort"/>
+                <param name="control_mode">velocity</param>
+            </joint>
+            <joint name="joint8">
+                <command_interface name="velocity"/>
+                <state_interface name="position">
+                  <param name="initial_value">0</param>
+                </state_interface>
+                <state_interface name="velocity"/>
+                <state_interface name="effort"/>
+                <param name="control_mode">velocity</param>
+            </joint>
+            <joint name="joint9">
+                <command_interface name="velocity"/>
+                <state_interface name="position">
+                  <param name="initial_value">0</param>
+                </state_interface>
+                <state_interface name="velocity"/>
+                <state_interface name="effort"/>
+                <param name="control_mode">velocity</param>
+            </joint>
         </ros2_control>
   </xacro:macro>
