Commit message: ros2 control for lekiwi (#1)

File: urdf/lekiwi.urdf (robot description, URDF)
Before this commit: robot LeKiwi, 45 links, 44 joints
Links:
- added link base_link
- link 4-Omni-Directional-Wheel_Single_Body-v1: geometry collision mesh filename=package://lekiwi/urdf/meshes/4-Omni-Directional-Wheel_Singl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 scale=0.001 0.001 0.001; visual mesh filename=package://lekiwi/urdf/meshes/4-Omni-Directional-Wheel_Singl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 scale=0.001 0.001 0.001
- link 4-Omni-Directional-Wheel_Single_Body-v1-1: geometry collision mesh filename=package://lekiwi/urdf/meshes/4-Omni-Directional-Wheel_Singl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 scale=0.001 0.001 0.001; visual mesh filename=package://lekiwi/urdf/meshes/4-Omni-Directional-Wheel_Singl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 scale=0.001 0.001 0.001
- link 4-Omni-Directional-Wheel_Single_Body-v1-2: geometry collision mesh filename=package://lekiwi/urdf/meshes/4-Omni-Directional-Wheel_Singl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 scale=0.001 0.001 0.001; visual mesh filename=package://lekiwi/urdf/meshes/4-Omni-Directional-Wheel_Singl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 scale=0.001 0.001 0.001
- link 94868A713_NO-THREADS_Female-Threaded-Hex-Standoff: geometry collision mesh filename=package://lekiwi/urdf/meshes/94868A713_NO-THREADS_Female-Th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 scale=0.001 0.001 0.001; visual mesh filename=package://lekiwi/urdf/meshes/94868A713_NO-THREADS_Female-Th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 scale=0.001 0.001 0.001
- link 94868A713_NO-THREADS_Female-Threaded-Hex-Standoff-1: geometry collision mesh filename=package://lekiwi/urdf/meshes/94868A713_NO-THREADS_Female-Th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 scale=0.001 0.001 0.001; visual mesh filename=package://lekiwi/urdf/meshes/94868A713_NO-THREADS_Female-Th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 scale=0.001 0.001 0.001
- link 94868A713_NO-THREADS_Female-Threaded-Hex-Standoff-2: geometry collision mesh filename=package://lekiwi/urdf/meshes/94868A713_NO-THREADS_Female-Th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 scale=0.001 0.001 0.001; visual mesh filename=package://lekiwi/urdf/meshes/94868A713_NO-THREADS_Female-Th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 scale=0.001 0.001 0.001
- link 94868A713_NO-THREADS_Female-Threaded-Hex-Standoff-3: geometry collision mesh filename=package://lekiwi/urdf/meshes/94868A713_NO-THREADS_Female-Th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 scale=0.001 0.001 0.001; visual mesh filename=package://lekiwi/urdf/meshes/94868A713_NO-THREADS_Female-Th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 scale=0.001 0.001 0.001
- link 94868A713_NO-THREADS_Female-Threaded-Hex-Standoff-4: geometry collision mesh filename=package://lekiwi/urdf/meshes/94868A713_NO-THREADS_Female-Th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 scale=0.001 0.001 0.001; visual mesh filename=package://lekiwi/urdf/meshes/94868A713_NO-THREADS_Female-Th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 scale=0.001 0.001 0.001
- link 94868A713_NO-THREADS_Female-Threaded-Hex-Standoff-5: geometry collision mesh filename=package://lekiwi/urdf/meshes/94868A713_NO-THREADS_Female-Th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 scale=0.001 0.001 0.001; visual mesh filename=package://lekiwi/urdf/meshes/94868A713_NO-THREADS_Female-Th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 scale=0.001 0.001 0.001
- link Base_08q-v1: geometry collision mesh filename=package://lekiwi/urdf/meshes/Base_08q-v1.stl scale=0.001 0.001 0.001; visual mesh filename=package://lekiwi/urdf/meshes/Base_08q-v1.stl scale=0.001 0.001 0.001
- link Battery---Battery-5.2-Ah-DC5521-Plug-v2: geometry collision mesh filename=package://lekiwi/urdf/meshes/Battery---Battery-5.2-Ah-DC552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 scale=0.001 0.001 0.001; visual mesh filename=package://lekiwi/urdf/meshes/Battery---Battery-5.2-Ah-DC552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 scale=0.001 0.001 0.001
- link Bottom-V2-v3: geometry collision mesh filename=package://lekiwi/urdf/meshes/Bottom-V2-v3.stl scale=0.001 0.001 0.001; visual mesh filename=package://lekiwi/urdf/meshes/Bottom-V2-v3.stl scale=0.001 0.001 0.001
- link Camera-Model-v3: geometry collision mesh filename=package://lekiwi/urdf/meshes/Camera-Model-v3.stl scale=0.001 0.001 0.001; visual mesh filename=package://lekiwi/urdf/meshes/Camera-Model-v3.stl scale=0.001 0.001 0.001
- link Camera-Model-v3-1: geometry collision mesh filename=package://lekiwi/urdf/meshes/Camera-Model-v3-1.stl scale=0.001 0.001 0.001; visual mesh filename=package://lekiwi/urdf/meshes/Camera-Model-v3-1.stl scale=0.001 0.001 0.001
- link Camera-Mount-v8: geometry collision mesh filename=package://lekiwi/urdf/meshes/Camera-Mount-v8.stl scale=0.001 0.001 0.001; visual mesh filename=package://lekiwi/urdf/meshes/Camera-Mount-v8.stl scale=0.001 0.001 0.001
- link Moving_Jaw_08d-v1: geometry collision mesh filename=package://lekiwi/urdf/meshes/Moving_Jaw_08d-v1.stl scale=0.001 0.001 0.001; visual mesh filename=package://lekiwi/urdf/meshes/Moving_Jaw_08d-v1.stl scale=0.001 0.001 0.001
- link Passive_Horn_01-v1: geometry collision mesh filename=package://lekiwi/urdf/meshes/Passive_Horn_01-v1.stl scale=0.001 0.001 0.001; visual mesh filename=package://lekiwi/urdf/meshes/Passive_Horn_01-v1.stl scale=0.001 0.001 0.001
- link Rotation_Pitch_08i-v1: geometry collision mesh filename=package://lekiwi/urdf/meshes/Rotation_Pitch_08i-v1.stl scale=0.001 0.001 0.001; visual mesh filename=package://lekiwi/urdf/meshes/Rotation_Pitch_08i-v1.stl scale=0.001 0.001 0.001
- link SO_ARM100_08k_116_Square-v1: geometry collision mesh filename=package://lekiwi/urdf/meshes/SO_ARM100_08k_116_Square-v1.stl scale=0.001 0.001 0.001; visual mesh filename=package://lekiwi/urdf/meshes/SO_ARM100_08k_116_Square-v1.stl scale=0.001 0.001 0.001
- link SO_ARM100_08k_Asym_Mirror_Clip-v1: geometry collision mesh filename=package://lekiwi/urdf/meshes/SO_ARM100_08k_Asym_Mirror_Clip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 scale=0.001 0.001 0.001; visual mesh filename=package://lekiwi/urdf/meshes/SO_ARM100_08k_Asym_Mirror_Clip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 scale=0.001 0.001 0.001
- link SO_ARM100_08k_Mirror-v1: geometry collision mesh filename=package://lekiwi/urdf/meshes/SO_ARM100_08k_Mirror-v1.stl scale=0.001 0.001 0.001; visual mesh filename=package://lekiwi/urdf/meshes/SO_ARM100_08k_Mirror-v1.stl scale=0.001 0.001 0.001
- link ST3215_Servo_Motor-v1: geometry collision mesh filename=package://lekiwi/urdf/meshes/ST3215_Servo_Motor-v1.stl scale=0.001 0.001 0.001; visual mesh filename=package://lekiwi/urdf/meshes/ST3215_Servo_Motor-v1.stl scale=0.001 0.001 0.001
- link ST3215_Servo_Motor-v1-1: geometry collision mesh filename=package://lekiwi/urdf/meshes/ST3215_Servo_Motor-v1-1.stl scale=0.001 0.001 0.001; visual mesh filename=package://lekiwi/urdf/meshes/ST3215_Servo_Motor-v1-1.stl scale=0.001 0.001 0.001
- link ST3215_Servo_Motor-v1-2: geometry collision mesh filename=package://lekiwi/urdf/meshes/ST3215_Servo_Motor-v1-2.stl scale=0.001 0.001 0.001; visual mesh filename=package://lekiwi/urdf/meshes/ST3215_Servo_Motor-v1-2.stl scale=0.001 0.001 0.001
- link STS3215_03a-v1: geometry collision mesh filename=package://lekiwi/urdf/meshes/STS3215_03a-v1.stl scale=0.001 0.001 0.001; visual mesh filename=package://lekiwi/urdf/meshes/STS3215_03a-v1.stl scale=0.001 0.001 0.001
- link STS3215_03a-v1-1: geometry collision mesh filename=package://lekiwi/urdf/meshes/STS3215_03a-v1-1.stl scale=0.001 0.001 0.001; visual mesh filename=package://lekiwi/urdf/meshes/STS3215_03a-v1-1.stl scale=0.001 0.001 0.001
- link STS3215_03a-v1-2: geometry collision mesh filename=package://lekiwi/urdf/meshes/STS3215_03a-v1-2.stl scale=0.001 0.001 0.001; visual mesh filename=package://lekiwi/urdf/meshes/STS3215_03a-v1-2.stl scale=0.001 0.001 0.001
- link STS3215_03a-v1-3: geometry collision mesh filename=package://lekiwi/urdf/meshes/STS3215_03a-v1-3.stl scale=0.001 0.001 0.001; visual mesh filename=package://lekiwi/urdf/meshes/STS3215_03a-v1-3.stl scale=0.001 0.001 0.001
- link STS3215_03a-v1-4: geometry collision mesh filename=package://lekiwi/urdf/meshes/STS3215_03a-v1-4.stl scale=0.001 0.001 0.001; visual mesh filename=package://lekiwi/urdf/meshes/STS3215_03a-v1-4.stl scale=0.001 0.001 0.001
- link STS3215_03a_Wrist_Roll-v1: geometry collision mesh filename=package://lekiwi/urdf/meshes/STS3215_03a_Wrist_Roll-v1.stl scale=0.001 0.001 0.001; visual mesh filename=package://lekiwi/urdf/meshes/STS3215_03a_Wrist_Roll-v1.stl scale=0.001 0.001 0.001
- link Top-V2-v2: geometry collision mesh filename=package://lekiwi/urdf/meshes/Top-V2-v2.stl scale=0.001 0.001 0.001; visual mesh filename=package://lekiwi/urdf/meshes/Top-V2-v2.stl scale=0.001 0.001 0.001
- link WaveShare_Mounting_Plate_01d-v1: geometry collision mesh filename=package://lekiwi/urdf/meshes/WaveShare_Mounting_Plate_01d-v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 scale=0.001 0.001 0.001; visual mesh filename=package://lekiwi/urdf/meshes/WaveShare_Mounting_Plate_01d-v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 scale=0.001 0.001 0.001
- link Wrist-Camera-Mount-v11: geometry collision mesh filename=package://lekiwi/urdf/meshes/Wrist-Camera-Mount-v11.stl scale=0.001 0.001 0.001; visual mesh filename=package://lekiwi/urdf/meshes/Wrist-Camera-Mount-v11.stl scale=0.001 0.001 0.001
- link Wrist_Roll_08c-v1: geometry collision mesh filename=package://lekiwi/urdf/meshes/Wrist_Roll_08c-v1.stl scale=0.001 0.001 0.001; visual mesh filename=package://lekiwi/urdf/meshes/Wrist_Roll_08c-v1.stl scale=0.001 0.001 0.001
- link Wrist_Roll_Pitch_08i-v1: geometry collision mesh filename=package://lekiwi/urdf/meshes/Wrist_Roll_Pitch_08i-v1.stl scale=0.001 0.001 0.001; visual mesh filename=package://lekiwi/urdf/meshes/Wrist_Roll_Pitch_08i-v1.stl scale=0.001 0.001 0.001
- link base_plate_layer1-v5: geometry collision mesh filename=package://lekiwi/urdf/meshes/base_plate_layer1-v5.stl scale=0.001 0.001 0.001; visual mesh filename=package://lekiwi/urdf/meshes/base_plate_layer1-v5.stl scale=0.001 0.001 0.001
- link base_plate_layer2-v3: geometry collision mesh filename=package://lekiwi/urdf/meshes/base_plate_layer2-v3.stl scale=0.001 0.001 0.001; visual mesh filename=package://lekiwi/urdf/meshes/base_plate_layer2-v3.stl scale=0.001 0.001 0.001
- link drive_motor_mount-v11: geometry collision mesh filename=package://lekiwi/urdf/meshes/drive_motor_mount-v11.stl scale=0.001 0.001 0.001; visual mesh filename=package://lekiwi/urdf/meshes/drive_motor_mount-v11.stl scale=0.001 0.001 0.001
- link drive_motor_mount-v11-1: geometry collision mesh filename=package://lekiwi/urdf/meshes/drive_motor_mount-v11-1.stl scale=0.001 0.001 0.001; visual mesh filename=package://lekiwi/urdf/meshes/drive_motor_mount-v11-1.stl scale=0.001 0.001 0.001
- link drive_motor_mount-v11-2: geometry collision mesh filename=package://lekiwi/urdf/meshes/drive_motor_mount-v11-2.stl scale=0.001 0.001 0.001; visual mesh filename=package://lekiwi/urdf/meshes/drive_motor_mount-v11-2.stl scale=0.001 0.001 0.001
- link lipo_battery_mount-v3: geometry collision mesh filename=package://lekiwi/urdf/meshes/lipo_battery_mount-v3.stl scale=0.001 0.001 0.001; visual mesh filename=package://lekiwi/urdf/meshes/lipo_battery_mount-v3.stl scale=0.001 0.001 0.001
- link omni_wheel_mount-v5: geometry collision mesh filename=package://lekiwi/urdf/meshes/omni_wheel_mount-v5.stl scale=0.001 0.001 0.001; visual mesh filename=package://lekiwi/urdf/meshes/omni_wheel_mount-v5.stl scale=0.001 0.001 0.001
- link omni_wheel_mount-v5-1: geometry collision mesh filename=package://lekiwi/urdf/meshes/omni_wheel_mount-v5-1.stl scale=0.001 0.001 0.001; visual mesh filename=package://lekiwi/urdf/meshes/omni_wheel_mount-v5-1.stl scale=0.001 0.001 0.001
- link omni_wheel_mount-v5-2: geometry collision mesh filename=package://lekiwi/urdf/meshes/omni_wheel_mount-v5-2.stl scale=0.001 0.001 0.001; visual mesh filename=package://lekiwi/urdf/meshes/omni_wheel_mount-v5-2.stl scale=0.001 0.001 0.001
- link servo_controller_mount-v3: geometry collision mesh filename=package://lekiwi/urdf/meshes/servo_controller_mount-v3.stl scale=0.001 0.001 0.001; visual mesh filename=package://lekiwi/urdf/meshes/servo_controller_mount-v3.stl scale=0.001 0.001 0.001
Joints:
- removed joint ST3215_Servo_Motor-v1-1_Revolute-62
- removed joint ST3215_Servo_Motor-v1-2_Revolute-60
- removed joint ST3215_Servo_Motor-v1_Revolute-64
- added joint base_mount: type fixed, parent base_link, child base_plate_layer1-v5, origin xyz=0.0 0.0 0.0 rpy=0.0 0.0 -1.5707963267948966
- added joint joint7: type continuous, parent ST3215_Servo_Motor-v1, child omni_wheel_mount-v5, origin xyz=0.010249999999999999 -0.010762340000000004 0.046859090000000006 rpy=-1.5707963267948966 1.5707963267948966 0, axis -0.866025 -2.0578792567370943e-32 0.5
- added joint joint8: type continuous, parent ST3215_Servo_Motor-v1-2, child omni_wheel_mount-v5-2, origin xyz=0.010249999999999999 -0.035199999999999995 -0.03275 rpy=-1.5707963267948966 1.5707963267948966 0, axis 0.0 0.0 -1.0
- added joint joint9: type continuous, parent ST3215_Servo_Motor-v1-1, child omni_wheel_mount-v5-1, origin xyz=0.010249999999999999 0.04636234 -0.014801910000000005 rpy=-1.5707963267948966 1.5707963267948966 0, axis 0.866025 1.0674582272562919e-32 0.5
- joint STS3215_03a-v1-1_Revolute-49: type continuous -> fixed
- joint STS3215_03a-v1-2_Revolute-51: type continuous -> fixed
- joint STS3215_03a-v1-3_Revolute-53: type continuous -> fixed
- joint STS3215_03a-v1-4_Revolute-57: type continuous -> fixed
- joint STS3215_03a-v1_Revolute-45: type continuous -> fixed
- joint STS3215_03a_Wrist_Roll-v1_Revolute-55: type continuous -> fixed
