Commit message: fixed issue with wheels. part of the problem was zombie node publishing weird commands

File: urdf/lekiwi.urdf (robot description, URDF)
Before this commit: robot LeKiwi, 46 links, 45 joints
Links:
- added link omni3_rim_joint7, mass 0.001; collision mesh filename=package://lekiwi/third_party/omni3ros_pkg/mesh/rim.stl scale=2.857142857 2.857142857 2.857142857; visual mesh filename=package://lekiwi/third_party/omni3ros_pkg/mesh/rim.stl scale=2.857142857 2.857142857 2.857142857
- added link omni3_rim_joint8, mass 0.001; collision mesh filename=package://lekiwi/third_party/omni3ros_pkg/mesh/rim.stl scale=2.857142857 2.857142857 2.857142857; visual mesh filename=package://lekiwi/third_party/omni3ros_pkg/mesh/rim.stl scale=2.857142857 2.857142857 2.857142857
- added link omni3_rim_joint9, mass 0.001; collision mesh filename=package://lekiwi/third_party/omni3ros_pkg/mesh/rim.stl scale=2.857142857 2.857142857 2.857142857; visual mesh filename=package://lekiwi/third_party/omni3ros_pkg/mesh/rim.stl scale=2.857142857 2.857142857 2.857142857
- added link omni3_roller_e_joint7, mass 0.002; collision mesh filename=package://lekiwi/third_party/omni3ros_pkg/mesh/roller.stl scale=2.857142857 2.857142857 2.857142857; visual mesh filename=package://lekiwi/third_party/omni3ros_pkg/mesh/roller.stl scale=2.857142857 2.857142857 2.857142857
- added link omni3_roller_e_joint8, mass 0.002; collision mesh filename=package://lekiwi/third_party/omni3ros_pkg/mesh/roller.stl scale=2.857142857 2.857142857 2.857142857; visual mesh filename=package://lekiwi/third_party/omni3ros_pkg/mesh/roller.stl scale=2.857142857 2.857142857 2.857142857
- added link omni3_roller_e_joint9, mass 0.002; collision mesh filename=package://lekiwi/third_party/omni3ros_pkg/mesh/roller.stl scale=2.857142857 2.857142857 2.857142857; visual mesh filename=package://lekiwi/third_party/omni3ros_pkg/mesh/roller.stl scale=2.857142857 2.857142857 2.857142857
- added link omni3_roller_n_joint7, mass 0.002; collision mesh filename=package://lekiwi/third_party/omni3ros_pkg/mesh/roller.stl scale=2.857142857 2.857142857 2.857142857; visual mesh filename=package://lekiwi/third_party/omni3ros_pkg/mesh/roller.stl scale=2.857142857 2.857142857 2.857142857
- added link omni3_roller_n_joint8, mass 0.002; collision mesh filename=package://lekiwi/third_party/omni3ros_pkg/mesh/roller.stl scale=2.857142857 2.857142857 2.857142857; visual mesh filename=package://lekiwi/third_party/omni3ros_pkg/mesh/roller.stl scale=2.857142857 2.857142857 2.857142857
- added link omni3_roller_n_joint9, mass 0.002; collision mesh filename=package://lekiwi/third_party/omni3ros_pkg/mesh/roller.stl scale=2.857142857 2.857142857 2.857142857; visual mesh filename=package://lekiwi/third_party/omni3ros_pkg/mesh/roller.stl scale=2.857142857 2.857142857 2.857142857
- added link omni3_roller_ne_joint7, mass 0.002; collision mesh filename=package://lekiwi/third_party/omni3ros_pkg/mesh/roller.stl scale=2.857142857 2.857142857 2.857142857; visual mesh filename=package://lekiwi/third_party/omni3ros_pkg/mesh/roller.stl scale=2.857142857 2.857142857 2.857142857
- added link omni3_roller_ne_joint8, mass 0.002; collision mesh filename=package://lekiwi/third_party/omni3ros_pkg/mesh/roller.stl scale=2.857142857 2.857142857 2.857142857; visual mesh filename=package://lekiwi/third_party/omni3ros_pkg/mesh/roller.stl scale=2.857142857 2.857142857 2.857142857
- added link omni3_roller_ne_joint9, mass 0.002; collision mesh filename=package://lekiwi/third_party/omni3ros_pkg/mesh/roller.stl scale=2.857142857 2.857142857 2.857142857; visual mesh filename=package://lekiwi/third_party/omni3ros_pkg/mesh/roller.stl scale=2.857142857 2.857142857 2.857142857
- added link omni3_roller_nw_joint7, mass 0.002; collision mesh filename=package://lekiwi/third_party/omni3ros_pkg/mesh/roller.stl scale=2.857142857 2.857142857 2.857142857; visual mesh filename=package://lekiwi/third_party/omni3ros_pkg/mesh/roller.stl scale=2.857142857 2.857142857 2.857142857
- added link omni3_roller_nw_joint8, mass 0.002; collision mesh filename=package://lekiwi/third_party/omni3ros_pkg/mesh/roller.stl scale=2.857142857 2.857142857 2.857142857; visual mesh filename=package://lekiwi/third_party/omni3ros_pkg/mesh/roller.stl scale=2.857142857 2.857142857 2.857142857
- added link omni3_roller_nw_joint9, mass 0.002; collision mesh filename=package://lekiwi/third_party/omni3ros_pkg/mesh/roller.stl scale=2.857142857 2.857142857 2.857142857; visual mesh filename=package://lekiwi/third_party/omni3ros_pkg/mesh/roller.stl scale=2.857142857 2.857142857 2.857142857
- added link omni3_roller_s_joint7, mass 0.002; collision mesh filename=package://lekiwi/third_party/omni3ros_pkg/mesh/roller.stl scale=2.857142857 2.857142857 2.857142857; visual mesh filename=package://lekiwi/third_party/omni3ros_pkg/mesh/roller.stl scale=2.857142857 2.857142857 2.857142857
- added link omni3_roller_s_joint8, mass 0.002; collision mesh filename=package://lekiwi/third_party/omni3ros_pkg/mesh/roller.stl scale=2.857142857 2.857142857 2.857142857; visual mesh filename=package://lekiwi/third_party/omni3ros_pkg/mesh/roller.stl scale=2.857142857 2.857142857 2.857142857
- added link omni3_roller_s_joint9, mass 0.002; collision mesh filename=package://lekiwi/third_party/omni3ros_pkg/mesh/roller.stl scale=2.857142857 2.857142857 2.857142857; visual mesh filename=package://lekiwi/third_party/omni3ros_pkg/mesh/roller.stl scale=2.857142857 2.857142857 2.857142857
- added link omni3_roller_se_joint7, mass 0.002; collision mesh filename=package://lekiwi/third_party/omni3ros_pkg/mesh/roller.stl scale=2.857142857 2.857142857 2.857142857; visual mesh filename=package://lekiwi/third_party/omni3ros_pkg/mesh/roller.stl scale=2.857142857 2.857142857 2.857142857
- added link omni3_roller_se_joint8, mass 0.002; collision mesh filename=package://lekiwi/third_party/omni3ros_pkg/mesh/roller.stl scale=2.857142857 2.857142857 2.857142857; visual mesh filename=package://lekiwi/third_party/omni3ros_pkg/mesh/roller.stl scale=2.857142857 2.857142857 2.857142857
- added link omni3_roller_se_joint9, mass 0.002; collision mesh filename=package://lekiwi/third_party/omni3ros_pkg/mesh/roller.stl scale=2.857142857 2.857142857 2.857142857; visual mesh filename=package://lekiwi/third_party/omni3ros_pkg/mesh/roller.stl scale=2.857142857 2.857142857 2.857142857
- added link omni3_roller_sw_joint7, mass 0.002; collision mesh filename=package://lekiwi/third_party/omni3ros_pkg/mesh/roller.stl scale=2.857142857 2.857142857 2.857142857; visual mesh filename=package://lekiwi/third_party/omni3ros_pkg/mesh/roller.stl scale=2.857142857 2.857142857 2.857142857
- added link omni3_roller_sw_joint8, mass 0.002; collision mesh filename=package://lekiwi/third_party/omni3ros_pkg/mesh/roller.stl scale=2.857142857 2.857142857 2.857142857; visual mesh filename=package://lekiwi/third_party/omni3ros_pkg/mesh/roller.stl scale=2.857142857 2.857142857 2.857142857
- added link omni3_roller_sw_joint9, mass 0.002; collision mesh filename=package://lekiwi/third_party/omni3ros_pkg/mesh/roller.stl scale=2.857142857 2.857142857 2.857142857; visual mesh filename=package://lekiwi/third_party/omni3ros_pkg/mesh/roller.stl scale=2.857142857 2.857142857 2.857142857
- added link omni3_roller_w_joint7, mass 0.002; collision mesh filename=package://lekiwi/third_party/omni3ros_pkg/mesh/roller.stl scale=2.857142857 2.857142857 2.857142857; visual mesh filename=package://lekiwi/third_party/omni3ros_pkg/mesh/roller.stl scale=2.857142857 2.857142857 2.857142857
- added link omni3_roller_w_joint8, mass 0.002; collision mesh filename=package://lekiwi/third_party/omni3ros_pkg/mesh/roller.stl scale=2.857142857 2.857142857 2.857142857; visual mesh filename=package://lekiwi/third_party/omni3ros_pkg/mesh/roller.stl scale=2.857142857 2.857142857 2.857142857
- added link omni3_roller_w_joint9, mass 0.002; collision mesh filename=package://lekiwi/third_party/omni3ros_pkg/mesh/roller.stl scale=2.857142857 2.857142857 2.857142857; visual mesh filename=package://lekiwi/third_party/omni3ros_pkg/mesh/roller.stl scale=2.857142857 2.857142857 2.857142857
- link 4-Omni-Directional-Wheel_Single_Body-v1: geometry 
- link 4-Omni-Directional-Wheel_Single_Body-v1-1: geometry 
- link 4-Omni-Directional-Wheel_Single_Body-v1-2: geometry 
Joints:
- added joint omni3_rim_joint7_mount: type fixed, parent 4-Omni-Directional-Wheel_Single_Body-v1, child omni3_rim_joint7, origin xyz=-0.013748155616372878 -0.007937504497239081 -5.773159728050814e-17 rpy=1.5707963267948974 -1.3089969389957468 2.094395102393195
- added joint omni3_rim_joint8_mount: type fixed, parent 4-Omni-Directional-Wheel_Single_Body-v1-2, child omni3_rim_joint8, origin xyz=7.450578487500081e-12 0.015874999999999986 6.661338147750939e-18 rpy=1.5707963267948966 0.26179938779914924 -1.0046485565123013e-33
- added joint omni3_rim_joint9_mount: type fixed, parent 4-Omni-Directional-Wheel_Single_Body-v1-1, child omni3_rim_joint9, origin xyz=0.013748155931950041 -0.007937495502761073 -2.2204460492503132e-17 rpy=-0.5235987755982988 -1.5707963267948963 0
- added joint omni3_roller_e_joint7_joint: type continuous, parent omni3_rim_joint7, child omni3_roller_e_joint7, origin xyz=0.038714286 0.0 0.015714286 rpy=-1.570796327 0 0, axis 0 0 1
- added joint omni3_roller_e_joint8_joint: type continuous, parent omni3_rim_joint8, child omni3_roller_e_joint8, origin xyz=0.038714286 0.0 0.015714286 rpy=-1.570796327 0 0, axis 0 0 1
- added joint omni3_roller_e_joint9_joint: type continuous, parent omni3_rim_joint9, child omni3_roller_e_joint9, origin xyz=0.038714286 0.0 0.015714286 rpy=-1.570796327 0 0, axis 0 0 1
- added joint omni3_roller_n_joint7_joint: type continuous, parent omni3_rim_joint7, child omni3_roller_n_joint7, origin xyz=0.0 0.038714286 0.015714286 rpy=-1.570796327 0 1.570796327, axis 0 0 1
- added joint omni3_roller_n_joint8_joint: type continuous, parent omni3_rim_joint8, child omni3_roller_n_joint8, origin xyz=0.0 0.038714286 0.015714286 rpy=-1.570796327 0 1.570796327, axis 0 0 1
- added joint omni3_roller_n_joint9_joint: type continuous, parent omni3_rim_joint9, child omni3_roller_n_joint9, origin xyz=0.0 0.038714286 0.015714286 rpy=-1.570796327 0 1.570796327, axis 0 0 1
- added joint omni3_roller_ne_joint7_joint: type continuous, parent omni3_rim_joint7, child omni3_roller_ne_joint7, origin xyz=0.027375134 0.027375134 -0.015714286 rpy=-1.570796327 0 0.785398163, axis 0 0 1
- added joint omni3_roller_ne_joint8_joint: type continuous, parent omni3_rim_joint8, child omni3_roller_ne_joint8, origin xyz=0.027375134 0.027375134 -0.015714286 rpy=-1.570796327 0 0.785398163, axis 0 0 1
- added joint omni3_roller_ne_joint9_joint: type continuous, parent omni3_rim_joint9, child omni3_roller_ne_joint9, origin xyz=0.027375134 0.027375134 -0.015714286 rpy=-1.570796327 0 0.785398163, axis 0 0 1
- added joint omni3_roller_nw_joint7_joint: type continuous, parent omni3_rim_joint7, child omni3_roller_nw_joint7, origin xyz=-0.027375134 0.027375134 -0.015714286 rpy=-1.570796327 0 2.356194490, axis 0 0 1
- added joint omni3_roller_nw_joint8_joint: type continuous, parent omni3_rim_joint8, child omni3_roller_nw_joint8, origin xyz=-0.027375134 0.027375134 -0.015714286 rpy=-1.570796327 0 2.356194490, axis 0 0 1
- added joint omni3_roller_nw_joint9_joint: type continuous, parent omni3_rim_joint9, child omni3_roller_nw_joint9, origin xyz=-0.027375134 0.027375134 -0.015714286 rpy=-1.570796327 0 2.356194490, axis 0 0 1
- added joint omni3_roller_s_joint7_joint: type continuous, parent omni3_rim_joint7, child omni3_roller_s_joint7, origin xyz=0.0 -0.038714286 0.015714286 rpy=-1.570796327 0 -1.570796327, axis 0 0 1
- added joint omni3_roller_s_joint8_joint: type continuous, parent omni3_rim_joint8, child omni3_roller_s_joint8, origin xyz=0.0 -0.038714286 0.015714286 rpy=-1.570796327 0 -1.570796327, axis 0 0 1
- added joint omni3_roller_s_joint9_joint: type continuous, parent omni3_rim_joint9, child omni3_roller_s_joint9, origin xyz=0.0 -0.038714286 0.015714286 rpy=-1.570796327 0 -1.570796327, axis 0 0 1
- added joint omni3_roller_se_joint7_joint: type continuous, parent omni3_rim_joint7, child omni3_roller_se_joint7, origin xyz=0.027375134 -0.027375134 -0.015714286 rpy=-1.570796327 0 -0.785398163, axis 0 0 1
- added joint omni3_roller_se_joint8_joint: type continuous, parent omni3_rim_joint8, child omni3_roller_se_joint8, origin xyz=0.027375134 -0.027375134 -0.015714286 rpy=-1.570796327 0 -0.785398163, axis 0 0 1
- added joint omni3_roller_se_joint9_joint: type continuous, parent omni3_rim_joint9, child omni3_roller_se_joint9, origin xyz=0.027375134 -0.027375134 -0.015714286 rpy=-1.570796327 0 -0.785398163, axis 0 0 1
- added joint omni3_roller_sw_joint7_joint: type continuous, parent omni3_rim_joint7, child omni3_roller_sw_joint7, origin xyz=-0.027375134 -0.027375134 -0.015714286 rpy=-1.570796327 0 -2.356194490, axis 0 0 1
- added joint omni3_roller_sw_joint8_joint: type continuous, parent omni3_rim_joint8, child omni3_roller_sw_joint8, origin xyz=-0.027375134 -0.027375134 -0.015714286 rpy=-1.570796327 0 -2.356194490, axis 0 0 1
- added joint omni3_roller_sw_joint9_joint: type continuous, parent omni3_rim_joint9, child omni3_roller_sw_joint9, origin xyz=-0.027375134 -0.027375134 -0.015714286 rpy=-1.570796327 0 -2.356194490, axis 0 0 1
- added joint omni3_roller_w_joint7_joint: type continuous, parent omni3_rim_joint7, child omni3_roller_w_joint7, origin xyz=-0.038714286 0.0 0.015714286 rpy=-1.570796327 0 3.141592654, axis 0 0 1
- added joint omni3_roller_w_joint8_joint: type continuous, parent omni3_rim_joint8, child omni3_roller_w_joint8, origin xyz=-0.038714286 0.0 0.015714286 rpy=-1.570796327 0 3.141592654, axis 0 0 1
- added joint omni3_roller_w_joint9_joint: type continuous, parent omni3_rim_joint9, child omni3_roller_w_joint9, origin xyz=-0.038714286 0.0 0.015714286 rpy=-1.570796327 0 3.141592654, axis 0 0 1

Commit message: small update urdf gripper frame position

File: urdf/lekiwi.urdf (robot description, URDF)
Before this commit: robot LeKiwi, 73 links, 72 joints
Joints:
- joint STS3215_03a_v1_4_Revolute_57: axis -2.74128770133849e-31 -0.9063079999999999 -0.422618 -> 0.0 0.0 1.0; origin xyz=-0.032799999999999996 -0.023912249999999986 0.027026410000000018 rpy=-1.5707963267948968 3.944304526105059e-31 -1.9721522630525295e-31 -> xyz=-0.032799999999999996 -0.023912249999999986 0.027026410000000018 rpy=-2.7052606678110185 0.0 0.0

Commit message: fix rviz and controllers

File: urdf/lekiwi.urdf (robot description, URDF)
Before this commit: robot LeKiwi, 73 links, 72 joints
Links:
- added link Center_of_Grip_EE
Joints:
- added joint Center_of_Grip_08d-v1_Rigid-58: type fixed, parent STS3215_03a-v1-4, child Center_of_Grip_EE, origin xyz=-0.012 -0.08212249999999986 -0.024026410000000018 rpy=-2.7052606678110185 0.0 0.0
